File: hardware/PCB/mainClockPCB/mainClockPCB/_autosave-mainClockPCB.kicad_sch (KiCad schematic)
At the start: 54 parts, among them IC1 ESP32-S3-WROOM-1-N16R2, IC2 SPX1117M3-L_TR, IC3 MCP7940N-I_P, IC4 PAM8904QJER, J1 USB_C_Receptacle_USB2.0_16P, J2 Conn_01x09_Socket, J3 Conn_01x02_Socket, SW1 SW_Push, SW2 SW_Push, SW3 SW_Push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

Commit message: clean up of display pins on main board schema
Connections:
- net ESP_3V3: no longer J2.5 (Pin_5)
- net GND: no longer J2.7 (Pin_7), U3.35 (MTMS/IO42)
- net at IC1.21 (IO13), IC1.4 (IO4): no longer J2.1 (Pin_1), J2.2 (Pin_2)
- net at IC1.20 (IO12): no longer J2.3 (Pin_3)
- net at IC1.33 (IO40): no longer J2.4 (Pin_4)
- net at IC1.7 (IO7): no longer J2.9 (Pin_9)
- new net +3V3: J2.5 (Pin_5)
- new net +5V: J2.7 (Pin_7)
- new net LIGHT_SENSOR: J2.9 (Pin_9)
- new net OE_PWM: J2.1 (Pin_1)
- new net RCLK: J2.4 (Pin_4)
- new net SERIAL: J2.2 (Pin_2)
- new net SRCLK: J2.3 (Pin_3)
Other:
- moved on the sheet: J2, U3
