File: hardware/PCB/mainClockPCB/mainClockPCB/mainClockPCB.kicad_pcb (KiCad board)
At the start: 4 copper layers, 223 x 50 mm, 69 parts, among them IC1 TMP275AIDR, IC2 SPX1117M3-L_TR, IC3 MCP7940N-I_P, IC4 PAM8904QJER, J1 USB_C_Receptacle_USB2.0_16P, J2 Conn_01x09_Socket, J3 Conn_01x02_Socket, J4 Conn_01x08, J5 Conn_01x09, J6 Conn_01x09, J7 Conn_01x05, J8 Conn_01x06, J9 Conn_01x05, SW1 SW_Push, SW2 SW_Push, U1 PEC11R-4320K-S0012, U2 USBLC6-2SC6, U3 ESP32-S3-WROOM-2, U4 74HC165, Y1 AB26T-32.768KHZ-6

Commit message: fixed PCB routing for JTAG and serial headers
Parts:
- J7: value Conn_01x05 -> Conn_01x04; footprint Connector_PinSocket_2.54mm:PinSocket_1x05_P2.54mm_Vertical -> Connector_PinSocket_2.54mm:PinSocket_1x04_P2.54mm_Vertical
- moved J7 0.26 mm to (129.0, 112.5)
Connections:
- J7 pad 1: ESP_3v3 -> GND
- J7 pad 4: +5V -> unconnected-(J7-Pin_4-Pad4)
- J8 pad 2: JTAG_MTCK -> JTAG_MTMS
- J8 pad 3: JTAG_MTDO -> JTAG_MTCK
- J8 pad 4: JTAG_MTDI -> JTAG_MTDO
- J8 pad 5: JTAG_MTMS -> JTAG_MTDI
Routing:
- net JTAG_MTMS: track 25.4 -> 37.0 mm
- net +5V: track 227.3 -> 225.5 mm
- net JTAG_MTDI: track 28.5 -> 27.0 mm
- net JTAG_MTDO: track 31.5 -> 30.2 mm
- net JTAG_MTCK: track 34.6 -> 33.6 mm
