File: hardware/PCB/mainClockPCB/mainClockPCB/mainClockPCB.kicad_pcb (KiCad board)
At the start: 4 copper layers, 223 x 50 mm, 69 parts, among them IC1 TMP275AIDR, IC2 SPX1117M3-L_TR, IC3 MCP7940N-I_P, IC4 PAM8904QJER, J1 USB_C_Receptacle_USB2.0_16P, J2 Conn_01x09_Socket, J3 Conn_01x02_Socket, J4 Conn_01x08, J5 Conn_01x09, J6 Conn_01x09, J7 Conn_01x04, J8 Conn_01x06, J9 Conn_01x05, SW1 SW_Push, SW2 SW_Push, U1 PEC11R-4320K-S0012, U2 USBLC6-2SC6, U3 ESP32-S3-WROOM-2, U4 74HC165, Y1 AB26T-32.768KHZ-6

Commit message: Adjusted expansion bay placement to reduce knob conflict
Parts:
- moved J5 4.26 mm to (230.5, 89.6)
- moved J6 4.26 mm to (180.5, 89.6)
Routing:
- net GPIO47: track 82.7 -> 72.6 mm
- net SCL: track 140.0 -> 135.8 mm
- net GPIO48: track 76.9 -> 72.7 mm
- net GPIO18: track 89.9 -> 85.6 mm
- net GPIO17: track 90.2 -> 85.9 mm
- net SDA: track 142.9 -> 138.6 mm
- net GPIO16: track 91.2 -> 87.0 mm
- net +5V: track 225.5 -> 221.9 mm
- net GPIO21: track 78.5 -> 82.0 mm
Other:
- board text added: "2026-07-26"
- board text added: "KiCAD 10.0"
- board text added: "REV B"
- board text removed: "2026-02-26"
- board text removed: "DISPLAY PINOUT INTENDED FOR: 12C-LTP-587HR REV D"
- board text removed: "KiCAD 9.0"
- board text removed: "REV A"

Commit message: logic updated for final display PCB
Other:
- board text added: "2026-07-20"
- board text removed: "2026-07-26"
Changed lines of the file:
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@@
 		)
 	)
-	(gr_text "2026-07-26"
+	(gr_text "2026-07-20"
 		(at 144.5 115.375 0)
 		(layer "F.SilkS")
