File: hardware/PCB/mainClockPCB/mainClockPCB/mainClockPCB.kicad_sch (KiCad schematic)
At the start: 62 parts, among them IC1 TMP275AIDR, IC2 SPX1117M3-L_TR, IC3 MCP7940N-I_P, IC4 PAM8904QJER, J1 USB_C_Receptacle_USB2.0_16P, J2 Conn_01x09_Socket, J3 Conn_01x02_Socket, J4 Conn_01x08, J5 Conn_01x09, J6 Conn_01x09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

Commit message: fixed PCB routing for JTAG and serial headers
Parts:
- J7: footprint (none) -> Connector_PinSocket_2.54mm:PinSocket_1x04_P2.54mm_Vertical
Changed lines of the file:
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@@
 			)
 		)
-		(property "Footprint" ""
+		(property "Footprint" "Connector_PinSocket_2.54mm:PinSocket_1x04_P2.54mm_Vertical"
 			(at 261.62 149.86 0)
 			(hide yes)
