File: hardware/PCB/mainClockPCB/mainClockPCB/mainClockPCB.kicad_sch (KiCad schematic)
At the start: 62 parts, among them IC1 TMP275AIDR, IC2 SPX1117M3-L_TR, IC3 MCP7940N-I_P, IC4 PAM8904QJER, J1 USB_C_Receptacle_USB2.0_16P, J2 Conn_01x09_Socket, J3 Conn_01x02_Socket, J4 Conn_01x08, J5 Conn_01x09, J6 Conn_01x09, J7 Conn_01x04, J8 Conn_01x06, J9 Conn_01x05, SW1 SW_Push, SW2 SW_Push, U1 PEC11R-4320K-S0012, U2 USBLC6-2SC6, U3 ESP32-S3-WROOM-2, U4 74HC165, Y1 AB26T-32.768KHZ-6

Commit message: PISO shift register button handling and schematic/BOM fixes
Parts:
- IC2: value SPX1117M3-L_TR -> SPX1117M3-L-3-3/TR
Connections:
- net BUTTON_SERIAL: now also U4.9 (Q7); no longer U4.10 (DS)
Changed lines of the file:
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@@
 	)
 	(no_connect
-		(at 135.89 44.45)
+		(at 119.38 148.59)
 	)
 	(no_connect
-		(at 217.17 160.02)
+		(at 135.89 44.45)
 	)
 	(no_connect
-		(at 93.98 148.59)
+		(at 217.17 160.02)
 	)
 	(no_connect
@@
 	(wire
 		(pts
+			(xy 93.98 148.59) (xy 90.17 148.59)
+		)
+		(stroke
+			(width 0)
+			(type default)
+		)
+	)
+	(wire
+		(pts
 			(xy 77.47 71.12) (xy 77.47 74.93)
 		)
@@
 	(wire
 		(pts
+			(xy 90.17 148.59) (xy 90.17 149.86)
+		)
+		(stroke
+			(width 0)
+			(type default)
+		)
+	)
+	(wire
+		(pts
 			(xy 171.45 76.2) (xy 173.99 76.2)
 		)
@@
 	(wire
 		(pts
-			(xy 119.38 148.59) (xy 139.7 148.59)
-		)
-		(stroke
-			(width 0)
-			(type default)
-		)
-	)
-	(wire
-		(pts
 			(xy 255.27 25.4) (xy 237.49 25.4)
 		)
@@
 		)
 	)
+	(global_label "BUTTON_SERIAL"
+		(shape input)
+		(at 90.17 149.86 270)
+		(fields_autoplaced yes)
+		(effects
+			(font
+				(size 0.762 0.762)
+			)
+			(justify right)
+		)
+		(property "Intersheetrefs" "${INTERSHEET_REFS}"
+			(at 90.17 160.3601 90)
+			(hide yes)
+			(show_name no)
+			(do_not_autoplace no)
+			(effects
+				(font
+					(size 1.27 1.27)
+				)
+				(justify right)
+			)
+		)
+	)
 	(global_label "JTAG_MTMS"
 		(shape input)
@@
 		)
 	)
-	(global_label "BUTTON_SERIAL"
-		(shape input)
-		(at 139.7 148.59 0)
-		(fields_autoplaced yes)
-		(effects
-			(font
-				(size 0.762 0.762)
-			)
-			(justify left)
-		)
-		(property "Intersheetrefs" "${INTERSHEET_REFS}"
-			(at 150.2001 148.59 0)
-			(hide yes)
-			(show_name no)
-			(do_not_autoplace no)
-			(effects
-				(font
-					(size 1.27 1.27)
-				)
-				(justify left)
-			)
-		)
-	)
 	(global_label "GPIO21"
 		(shape input)
@@
 			)
 		)
-		(property "Value" "SPX1117M3-L_TR"
+		(property "Value" "SPX1117M3-L-3-3/TR"
 			(at 62.23 97.79 0)
 			(show_name no)
